File: main_pcb.sch (KiCad schematic (older format))
At the start: 21 parts

Commit message: add power supply on usb
Parts:
- added C? (x2): 100n, symbol Device:C_Small
- added J?: USB_conn, symbol LoRaWAN_lib:USB_conn
- added R? (x2): 22, symbol Device:R
- added R?: 5K, symbol Device:R
- added U?: USBLC6-2SC6, Package_TO_SOT_SMD:SOT-23-6, symbol Power_Protection:USBLC6-2SC6
- added U?: AMS1117-3.3, Package_TO_SOT_SMD:SOT-223-3_TabPin2, symbol Regulator_Linear:AMS1117-3.3
Connections:
- wire segments 100 -> 143

Commit message: add STLink connector
Parts:
- removed J?: Conn_01x05_Male, symbol Connector:Conn_01x05_Male
- added J?: STLink_conn, symbol LoRaWAN_lib:STLink_conn
Connections:
- wire segments 143 -> 145
Changed lines of the file:
@@
 Text Label 2500 6650 2    50   ~ 0
 BOOT1
-$Comp
-L Connector:Conn_01x05_Male J?
-U 1 1 5E493377
-P 1300 5800
-F 0 "J?" H 1150 5800 50  0000 R CNN
-F 1 "Conn_01x05_Male" V 1200 6100 50  0000 R CNN
-F 2 "" H 1300 5800 50  0001 C CNN
-F 3 "~" H 1300 5800 50  0001 C CNN
-	1    1300 5800
-	0    -1   -1   0
-$EndComp
-$Comp
-L power:VCC #PWR?
-U 1 1 5E49340B
-P 1100 5450
-F 0 "#PWR?" H 1100 5300 50  0001 C CNN
-F 1 "VCC" H 1117 5623 50  0000 C CNN
-F 2 "" H 1100 5450 50  0001 C CNN
-F 3 "" H 1100 5450 50  0001 C CNN
-	1    1100 5450
-	1    0    0    -1
-$EndComp
-Wire Wire Line
-	1100 5600 1100 5450
-Wire Wire Line
-	1200 5600 1200 5350
-Wire Wire Line
-	1300 5600 1300 5350
-Wire Wire Line
-	1400 5600 1400 5350
-$Comp
-L power:GND #PWR?
-U 1 1 5E4A87D6
-P 1500 5450
-F 0 "#PWR?" H 1500 5200 50  0001 C CNN
-F 1 "GND" H 1505 5277 50  0000 C CNN
-F 2 "" H 1500 5450 50  0001 C CNN
-F 3 "" H 1500 5450 50  0001 C CNN
-	1    1500 5450
-	-1   0    0    1
-$EndComp
-Wire Wire Line
-	1500 5600 1500 5450
-Text Label 1200 5350 3    50   ~ 0
-DIO
-Text Label 1300 5350 3    50   ~ 0
-DCLK
-Text Label 1400 5350 3    50   ~ 0
-R
 Wire Wire Line
 	8200 4350 8500 4350
@@
 	1    0    0    -1
 $EndComp
-$Comp
-L Power_Protection:USBLC6-2SC6 U?
-U 1 1 5E530E7D
-P 9700 4150
-F 0 "U?" H 9950 4550 50  0000 C CNN
-F 1 "USBLC6-2SC6" H 9300 4550 50  0000 C CNN
-F 2 "Package_TO_SOT_SMD:SOT-23-6" H 8950 4550 50  0001 C CNN
-F 3 "http://www2.st.com/resource/en/datasheet/CD00050750.pdf" H 9900 4500 50  0001 C CNN
-	1    9700 4150
-	1    0    0    -1
-$EndComp
 Wire Wire Line
 	10450 2800 10450 3000
@@
 Wire Wire Line
 	8850 4150 8200 4150
-Wire Wire Line
-	9700 3350 9700 3650
-$Comp
-L power:VCC #PWR?
-U 1 1 5E520873
-P 9700 3350
-F 0 "#PWR?" H 9700 3200 50  0001 C CNN
-F 1 "VCC" H 9717 3523 50  0000 C CNN
-F 2 "" H 9700 3350 50  0001 C CNN
-F 3 "" H 9700 3350 50  0001 C CNN
-	1    9700 3350
-	1    0    0    -1
-$EndComp
 $Comp
 L Regulator_Linear:AMS1117-3.3 U?
@@
 	10350 2800 10350 2900
 Wire Wire Line
-	10350 2900 9300 2900
+	10350 2900 9700 2900
 Wire Wire Line
 	9300 2900 9300 2350
@@
 Wire Wire Line
 	9600 2350 9750 2350
+$Comp
+L Power_Protection:USBLC6-2SC6 U?
+U 1 1 5E530E7D
+P 9700 4150
+F 0 "U?" H 9950 4550 50  0000 C CNN
+F 1 "USBLC6-2SC6" H 9300 4550 50  0000 C CNN
+F 2 "Package_TO_SOT_SMD:SOT-23-6" H 8950 4550 50  0001 C CNN
+F 3 "http://www2.st.com/resource/en/datasheet/CD00050750.pdf" H 9900 4500 50  0001 C CNN
+	1    9700 4150
+	1    0    0    -1
+$EndComp
+Wire Wire Line
+	9700 3650 9700 2900
+Connection ~ 9700 2900
+Wire Wire Line
+	9700 2900 9300 2900
+$Comp
+L power:GND #PWR?
+U 1 1 5E5F5DB3
+P 2450 6000
+F 0 "#PWR?" H 2450 5750 50  0001 C CNN
+F 1 "GND" V 2455 5872 50  0000 R CNN
+F 2 "" H 2450 6000 50  0001 C CNN
+F 3 "" H 2450 6000 50  0001 C CNN
+	1    2450 6000
+	0    -1   -1   0
+$EndComp
+Wire Wire Line
+	2000 6000 2450 6000
+Wire Wire Line
+	2000 5900 2450 5900
+Wire Wire Line
+	2000 5800 2450 5800
+$Comp
+L power:VCC #PWR?
+U 1 1 5E605111
+P 2450 5600
+F 0 "#PWR?" H 2450 5450 50  0001 C CNN
+F 1 "VCC" H 2467 5773 50  0000 C CNN
+F 2 "" H 2450 5600 50  0001 C CNN
+F 3 "" H 2450 5600 50  0001 C CNN
+	1    2450 5600
+	1    0    0    -1
+$EndComp
+Wire Wire Line
+	2450 5600 2450 5700
+Wire Wire Line
+	2450 5700 2000 5700
+Wire Wire Line
+	2000 6100 2450 6100
+Text Label 2450 6100 0    50   ~ 0
+R
+Text Label 2450 5900 0    50   ~ 0
+DCLK
+Text Label 2450 5800 0    50   ~ 0
+DIO
+$Comp
+L LoRaWAN_lib:STLink_conn J?
+U 1 1 5E61F628
+P 1750 5900
+F 0 "J?" H 1806 6325 50  0000 C CNN
+F 1 "STLink_conn" H 1806 6234 50  0000 C CNN
+F 2 "" H 1750 5900 50  0001 C CNN
+F 3 "" H 1750 5900 50  0001 C CNN
+	1    1750 5900
+	1    0    0    -1
+$EndComp
 $EndSCHEMATC

Commit message: home pc - add connectors for fw upgrade, power supplay connector, ant connector
Parts:
- added D? (x2): Blue, symbol Device:LED
- added J?: Conn_01x04_Male, symbol Connector:Conn_01x04_Male
- added J? (x3): Conn_01x03_Male, symbol Connector:Conn_01x03_Male
- added J?: Conn_Coaxial, symbol Connector:Conn_Coaxial
- added J? (x2): Conn_01x02_Female, symbol Connector:Conn_01x02_Female
- added J?: Conn_02x03_Top_Bottom, symbol Connector_Generic:Conn_02x03_Top_Bottom
- added R? (x4): 22, symbol Device:R
- added R?: 0, symbol Device:R
- added R? (x3): 510, symbol Device:R
- added SW?: SW_Push, symbol Switch:SW_Push
- D?: symbol RF_Module:RHF78-052 -> main_pcb-rescue:RHF78-052-RF_Module
- J?: symbol LoRaWAN_lib:USB_conn -> main_pcb-rescue:USB_conn-LoRaWAN_lib
- J?: symbol LoRaWAN_lib:STLink_conn -> main_pcb-rescue:STLink_conn-LoRaWAN_lib
Connections:
- net labels added: 3v3_STLink, AMS1117_3v3, RX_fw, TX_fw, UART_FW, USART2_RX, USART2_TX
- net labels removed: DCLK, DIO
- wire segments 145 -> 227
Other:
- moved on the sheet: J?

Commit message: add i2c, spi interface
Parts:
- added J?: Conn_01x03_Male, symbol Connector:Conn_01x03_Male
- added J? (x2): Conn_01x01_Male, symbol Connector:Conn_01x01_Male
- added J?: Conn_01x06_Male, symbol Connector:Conn_01x06_Male
- added J?: Conn_01x08_Male, symbol Connector:Conn_01x08_Male
- added R?: R_Variable, symbol Device:R_Variable
- added R? (x2): 10K, symbol Device:R
- added U?: DS2482-100, Housings_SOIC:SOIC-8_3.9x4.9mm_Pitch1.27mm, symbol lib:DS2482-100
Connections:
- net labels added: gpio, i2c1_scl, i2c1_sda, spi1_miso, spi1_mosi, spi1_nss, spi1_sck
- wire segments 227 -> 292
- no-connect marks 0 -> 14

Commit message: add RHF78 footprint
Parts:
- removed J?: Conn_01x08_Male, symbol Connector:Conn_01x08_Male
- added J13: Conn_01x09_Male, symbol Connector:Conn_01x09_Male
- U2: renamed from U?; symbol lib:DS2482-100 -> main_pcb-rescue:DS2482-100-lib
- gave numbers to parts that had none: 55
Connections:
- wire segments 292 -> 296
- no-connect marks 14 -> 15

Commit message: add footprint
Parts:
- removed J11, J12: Conn_01x02_Female, symbol Connector:Conn_01x02_Female
- added J11: Conn_02x02_Odd_Even, Pin_Headers:Pin_Header_Straight_2x02_Pitch2.54mm, symbol Connector_Generic:Conn_02x02_Odd_Even
- C1, C2, C3, C4, C5, C6, C7, C8, C9: footprint (none) -> Capacitors_SMD:C_0805_HandSoldering
- D1, D3, D4, D5: footprint (none) -> LEDs:LED_0805_HandSoldering
- D2: footprint (none) -> RHF78_footprint:RHF78_052
- J1: footprint (none) -> Pin_Headers:Pin_Header_Straight_1x05_Pitch2.54mm
- J10, J6, J7: footprint (none) -> Pin_Headers:Pin_Header_Straight_1x03_Pitch2.54mm
- J12: renamed from J13; footprint (none) -> Pin_Headers:Pin_Header_Straight_1x09_Pitch2.54mm; symbol Connector:Conn_01x09_Male -> main_pcb-rescue:Conn_01x09_Male-Connector
- J13: renamed from J14; footprint (none) -> U_FL:U_FL_smd
- J14: renamed from J15; footprint (none) -> Pin_Headers:Pin_Header_Straight_1x03_Pitch2.54mm
- J15: renamed from J16; footprint (none) -> Connectors:USB_Micro-B
- J2: footprint (none) -> Pin_Headers:Pin_Header_Straight_1x04_Pitch2.54mm
- J3, J4: footprint (none) -> Pin_Headers:Pin_Header_Straight_2x03_Pitch2.54mm
- J5, J9: footprint (none) -> Pin_Headers:Pin_Header_Straight_1x01_Pitch2.54mm
- J8: footprint (none) -> Pin_Headers:Pin_Header_Straight_1x06_Pitch2.54mm
- R1, R10, R11, R12, R13, R14, R15, R16, R18, R19, R2, R3, R4, R5, R6, R7, R8, R9: footprint (none) -> Resistors_SMD:R_0805_HandSoldering
- R17: footprint (none) -> Potentiometers:Potentiometer_Trimmer_Bourns_3296W
- U1: footprint Package_QFP:LQFP-48_7x7mm_P0.5mm -> Housings_QFP:LQFP-48_7x7mm_Pitch0.5mm
- U3: footprint Package_TO_SOT_SMD:SOT-23-6 -> TO_SOT_Packages_SMD:SOT-23-6_Handsoldering
- U4: footprint Package_TO_SOT_SMD:SOT-223-3_TabPin2 -> TO_SOT_Packages_SMD:SOT-223-3_TabPin2
- Y1: footprint (none) -> Crystals:Crystal_HC18-U_Vertical
- Y2: footprint (none) -> Crystals:Crystal_AT310_d3.0mm_l10.0mm_Vertical
Connections:
- net at D2.30 (RFIO_HF): now also J11.3 (Pin_3)
- net at D2.32 (RFIO_LF): now also J11.1 (Pin_1)
- net at R9.2: now also J11.2 (Pin_2), J11.4 (Pin_4)

Commit message: add key Reset footprint
Parts:
- J13: footprint U_FL:U_FL_smd -> U_FL_smd:U_FL_smd
- SW1, SW2: footprint (none) -> Button_Switch_SMD:SW_SPST_EVQPE1
Changed lines of the file:
@@
 EESchema Schematic File Version 4
-EELAYER 30 0
+LIBS:main_pcb-cache
+EELAYER 26 0
 EELAYER END
 $Descr A4 11693 8268
@@
 F 0 "SW2" V 6104 7048 50  0000 L CNN
 F 1 "Reset" V 6195 7048 50  0000 L CNN
-F 2 "" H 6150 6950 50  0001 C CNN
+F 2 "Button_Switch_SMD:SW_SPST_EVQPE1" H 6150 6950 50  0001 C CNN
 F 3 "" H 6150 6950 50  0001 C CNN
 	1    6150 6950
@@
 F 0 "J13" H 5900 725 50  0000 L CNN
 F 1 "Conn_Coaxial" H 5900 634 50  0000 L CNN
-F 2 "U_FL:U_FL_smd" H 5800 750 50  0001 C CNN
+F 2 "U_FL_smd:U_FL_smd" H 5800 750 50  0001 C CNN
 F 3 " ~" H 5800 750 50  0001 C CNN
 	1    5800 750
@@
 F 0 "SW1" H 1650 4135 50  0000 C CNN
 F 1 "SW_Push" H 1650 4044 50  0000 C CNN
-F 2 "" H 1650 4050 50  0001 C CNN
+F 2 "Button_Switch_SMD:SW_SPST_EVQPE1" H 1650 4050 50  0001 C CNN
 F 3 "~" H 1650 4050 50  0001 C CNN
 	1    1650 3850

Commit message: pcbnew
Parts:
- SW1, SW2: footprint Button_Switch_SMD:SW_SPST_EVQPE1 -> Buttons_Switches_SMD:SW_SPST_EVQPE1
Changed lines of the file:
@@
 EESchema Schematic File Version 4
-LIBS:main_pcb-cache
-EELAYER 26 0
+EELAYER 30 0
 EELAYER END
 $Descr A4 11693 8268
@@
 F 0 "SW2" V 6104 7048 50  0000 L CNN
 F 1 "Reset" V 6195 7048 50  0000 L CNN
-F 2 "Button_Switch_SMD:SW_SPST_EVQPE1" H 6150 6950 50  0001 C CNN
+F 2 "Buttons_Switches_SMD:SW_SPST_EVQPE1" H 6150 6950 50  0001 C CNN
 F 3 "" H 6150 6950 50  0001 C CNN
 	1    6150 6950
@@
 F 0 "SW1" H 1650 4135 50  0000 C CNN
 F 1 "SW_Push" H 1650 4044 50  0000 C CNN
-F 2 "Button_Switch_SMD:SW_SPST_EVQPE1" H 1650 4050 50  0001 C CNN
+F 2 "Buttons_Switches_SMD:SW_SPST_EVQPE1" H 1650 4050 50  0001 C CNN
 F 3 "~" H 1650 4050 50  0001 C CNN
 	1    1650 3850
