File: main_pcb.sch (KiCad schematic (older format))
At the start: 53 parts, among them J1 STLink_conn, J11 Conn_02x02_Odd_Even, J12 Conn_01x01_Male, J13 Conn_Coaxial, J14 Conn_01x03_Male, J15 USB_conn, J2 Conn_01x04_Male, J3 Conn_02x03_Odd_Even, J4 Conn_01x03_Male, J5 Conn_01x01_Male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

Commit message: pcbnew complited
Parts:
- D2: value RHF78-052 -> RHF78-052-RF_Module
Changed lines of the file:
@@
 P 3250 2650
 F 0 "D2" H 3275 3475 50  0000 C CNN
-F 1 "RHF78-052" H 3275 3384 50  0000 C CNN
+F 1 "RHF78-052-RF_Module" H 3275 3384 50  0000 C CNN
 F 2 "LoraWAN_pcb:RHF78_052" H 3150 2650 50  0001 C CNN
 F 3 "" H 3150 2650 50  0001 C CNN
