File: main_pcb.kicad_pcb (KiCad board)
At the start: 2 copper layers, 56 parts, among them J1 STLink_conn, J10 Conn_01x03_Male, J11 Conn_02x02_Odd_Even, J12 Conn_01x09_Male, J13 Conn_Coaxial, J14 Conn_01x03_Male, J15 USB_conn, J2 Conn_01x04_Male, J3 Conn_02x03_Top_Bottom, J4 Conn_02x03_Top_Bottom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

Commit message: center
Parts:
- C4, C5, R14, R15, R6, R7, U2: moved to B.Cu
- R11, Y1: moved to F.Cu
- moved U4 111.2 mm to (189.9, 90.7)
- moved R1 83.5 mm to (171.7, 82.5)
- moved R4 78.0 mm to (176.9, 78.6), turned to 0 degrees
- moved R2 75.4 mm to (165.3, 89.6), turned to 0 degrees
- moved C7 73.4 mm to (177.3, 87.0)
- moved J4 64.5 mm to (171.2, 121.4), turned to 0 degrees
- moved U2 64.3 mm to (121.5, 87.0), turned to 180 degrees
- moved D5 57.3 mm to (155.2, 95.8)
- moved R14 52.0 mm to (127.5, 87.2), turned to 90 degrees
- moved J6 51.7 mm to (101.8, 90.1), turned to 90 degrees
- moved J8 50.8 mm to (113.6, 59.7)
- moved R15 50.0 mm to (115.9, 86.8), turned to 90 degrees
- moved J3 49.7 mm to (124.6, 135.9), turned to 0 degrees
- moved R18 48.2 mm to (171.7, 85.4), turned to 0 degrees
- moved J7 47.2 mm to (101.8, 93.7), turned to 90 degrees
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Connections:
- R2 pad 2: Net-(J2-Pad2) -> Net-(J2-Pad3)
- R3 pad 2: Net-(J2-Pad3) -> Net-(J2-Pad2)
- U1 pad 25: Net-(J12-Pad5) -> Net-(J12-Pad8)
- U1 pad 26: Net-(J12-Pad6) -> Net-(J12-Pad7)
- U1 pad 27: Net-(J12-Pad7) -> Net-(J12-Pad6)
- U1 pad 28: Net-(J12-Pad8) -> Net-(J12-Pad5)
- U1 pad 45: Net-(J12-Pad1) -> Net-(J12-Pad2)
- U1 pad 46: Net-(J12-Pad2) -> Net-(J12-Pad1)
Routing:
- net GND: track 0.00 -> 90.0 mm, vias 0 -> 3
- net VCC: track 0.00 -> 40.8 mm
- net Net-(D2-Pad23): track 0.00 -> 38.2 mm, vias 0 -> 1
- net Net-(J12-Pad1): track 0.00 -> 37.5 mm
- net Net-(D2-Pad22): track 0.00 -> 36.1 mm, vias 0 -> 1
- net Net-(C4-Pad1): track 0.00 -> 34.6 mm, vias 0 -> 1
- net Net-(J14-Pad2): track 0.00 -> 33.0 mm
- net Net-(C5-Pad1): track 0.00 -> 28.8 mm, vias 0 -> 1
- net Net-(C2-Pad1): track 0.00 -> 20.1 mm
- net Net-(C3-Pad1): track 0.00 -> 14.3 mm
- net /i2c1_scl: track 0.00 -> 13.8 mm
- net /i2c1_sda: track 0.00 -> 13.5 mm
- net /spi1_nss: track 0.00 -> 13.1 mm
- net /spi1_mosi: track 0.00 -> 13.1 mm
- net /spi1_sck: track 0.00 -> 12.3 mm
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
Commit message: work PC
Parts:
- J3: value Conn_02x03_Top_Bottom -> Conn_02x03_Odd_Even; footprint Pin_Headers:Pin_Header_Straight_2x03_Pitch2.54mm -> Connector_PinHeader_2.54mm:PinHeader_2x03_P2.54mm_Vertical
- moved R2 62.4 mm to (105.9, 70.6), turned to 90 degrees
- moved R4 56.0 mm to (124.1, 97.0), turned to 90 degrees
- moved J3 32.2 mm to (110.5, 106.9), turned to 270 degrees
- moved R3 31.9 mm to (110.1, 72.0), turned to 90 degrees
- moved SW1 14.5 mm to (116.2, 99.4)
- moved J1 13.4 mm to (110.1, 97.8), turned to 270 degrees
- moved J10 9.75 mm to (102.4, 87.7), turned to 0 degrees
- moved J7 6.92 mm to (105.0, 87.6), turned to 0 degrees
- moved J6 6.48 mm to (107.7, 87.7), turned to 0 degrees
- moved D3 6.25 mm to (144.1, 75.9), turned to 180 degrees
- moved D1 4.42 mm to (122.7, 101.3), turned to 180 degrees
- moved J2 2.88 mm to (99.9, 109.3), turned to 180 degrees
Connections:
- J3 pad 2: VCC -> /3v3_STLink
- J3 pad 4: /3v3_STLink -> /AMS1117_3v3
- J3 pad 5: /AMS1117_3v3 -> VCC
Routing:
- net Net-(J2-Pad3): track 0.00 -> 49.7 mm
- net Net-(J2-Pad2): track 0.00 -> 46.1 mm
- net /R: track 0.00 -> 24.3 mm, vias 0 -> 1
- net VCC: track 40.8 -> 59.6 mm
- net /3v3_STLink: track 0.00 -> 14.4 mm
- net Net-(J1-Pad5): track 0.00 -> 12.9 mm
- net Net-(J1-Pad2): track 0.00 -> 8.68 mm
- net /RX_fw: track 0.00 -> 7.71 mm
- net Net-(D2-Pad13): track 0.00 -> 6.90 mm
- net Net-(D2-Pad12): track 0.00 -> 6.68 mm
- net Net-(D2-Pad14): track 0.00 -> 6.45 mm
- net GND: track 90.0 -> 95.7 mm
- net /UART_FW: track 0.00 -> 5.51 mm
- net Net-(J1-Pad3): track 0.00 -> 5.09 mm
- net Net-(D2-Pad16): track 0.00 -> 4.47 mm
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
Commit message: work PC
Parts:
- J4: value Conn_02x03_Top_Bottom -> Conn_02x03_Odd_Even; footprint Pin_Headers:Pin_Header_Straight_2x03_Pitch2.54mm -> Connector_PinHeader_2.54mm:PinHeader_2x03_P2.54mm_Vertical
- moved J4 44.9 mm to (126.6, 115.7)
- moved R5 32.5 mm to (144.5, 74.1), turned to 180 degrees
- moved D4 21.0 mm to (145.1, 86.9)
- moved R8 9.96 mm to (140.8, 88.7), turned to 270 degrees
- moved D3 6.44 mm to (150.3, 74.1), turned to 0 degrees
Connections:
- J4 pad 2: /BOOT0 -> VCC
- J4 pad 3: GND -> /BOOT0
- J4 pad 4: VCC -> /BOOT1
- J4 pad 5: /BOOT1 -> GND
Routing:
- net GND: track 95.7 -> 102.2 mm
- net Net-(D2-Pad21): track 0.00 -> 4.10 mm
- net Net-(D4-Pad1): track 0.00 -> 3.21 mm
- net Net-(D3-Pad1): track 0.00 -> 3.13 mm

Commit message: stm32 is bootom, rhf78 is top
Parts:
- J3, J4: footprint Connector_PinHeader_2.54mm:PinHeader_2x03_P2.54mm_Vertical -> Pin_Headers:Pin_Header_Straight_2x03_Pitch2.54mm
Changed lines of the file:
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@@
   )
   (setup
-    (last_trace_width 0.5)
+    (last_trace_width 0.25)
     (user_trace_width 0.5)
     (trace_clearance 0.2)
@@
     )
   )
-  (module Connector_PinHeader_2.54mm:PinHeader_2x03_P2.54mm_Vertical (layer F.Cu)
+  (module Pin_Headers:Pin_Header_Straight_2x03_Pitch2.54mm (layer F.Cu)
     (at 110.49 106.934 270)
     (descr "Through hole straight pin header, 2x03, 2.54mm pitch, double rows")
@@
     (pad 6 thru_hole oval (at 2.54 5.08 270) (size 1.7 1.7) (drill 1) (layers *.Cu *.Mask)
       (net 45 /UART_FW))
-    (model ${KISYS3DMOD}/Connector_PinHeader_2.54mm.3dshapes/PinHeader_2x03_P2.54mm_Vertical.wrl
-      (at (xyz 0 0 0))
-      (scale (xyz 1 1 1))
-      (rotate (xyz 0 0 0))
-    )
-  )
-  (module Connector_PinHeader_2.54mm:PinHeader_2x03_P2.54mm_Vertical (layer F.Cu)
+    (model ${KISYS3DMOD}/Pin_Headers.3dshapes/Pin_Header_Straight_2x03_Pitch2.54mm.wrl
+      (at (xyz 0 0 0))
+      (scale (xyz 1 1 1))
+      (rotate (xyz 0 0 0))
+    )
+  )
+  (module Pin_Headers:Pin_Header_Straight_2x03_Pitch2.54mm (layer F.Cu)
     (at 126.619 115.697)
     (descr "Through hole straight pin header, 2x03, 2.54mm pitch, double rows")
@@
       (effects (font (size 1 1) (thickness 0.15)))
     )
+    (fp_text user %R (at 1.27 2.54 90) (layer F.Fab)
+      (effects (font (size 1 1) (thickness 0.15)))
+    )
+    (fp_line (start 4.35 -1.8) (end -1.8 -1.8) (layer F.CrtYd) (width 0.05))
+    (fp_line (start 4.35 6.85) (end 4.35 -1.8) (layer F.CrtYd) (width 0.05))
+    (fp_line (start -1.8 6.85) (end 4.35 6.85) (layer F.CrtYd) (width 0.05))
+    (fp_line (start -1.8 -1.8) (end -1.8 6.85) (layer F.CrtYd) (width 0.05))
+    (fp_line (start -1.33 -1.33) (end 0 -1.33) (layer F.SilkS) (width 0.12))
+    (fp_line (start -1.33 0) (end -1.33 -1.33) (layer F.SilkS) (width 0.12))
+    (fp_line (start 1.27 -1.33) (end 3.87 -1.33) (layer F.SilkS) (width 0.12))
+    (fp_line (start 1.27 1.27) (end 1.27 -1.33) (layer F.SilkS) (width 0.12))
+    (fp_line (start -1.33 1.27) (end 1.27 1.27) (layer F.SilkS) (width 0.12))
+    (fp_line (start 3.87 -1.33) (end 3.87 6.41) (layer F.SilkS) (width 0.12))
+    (fp_line (start -1.33 1.27) (end -1.33 6.41) (layer F.SilkS) (width 0.12))
+    (fp_line (start -1.33 6.41) (end 3.87 6.41) (layer F.SilkS) (width 0.12))
+    (fp_line (start -1.27 0) (end 0 -1.27) (layer F.Fab) (width 0.1))
+    (fp_line (start -1.27 6.35) (end -1.27 0) (layer F.Fab) (width 0.1))
+    (fp_line (start 3.81 6.35) (end -1.27 6.35) (layer F.Fab) (width 0.1))
+    (fp_line (start 3.81 -1.27) (end 3.81 6.35) (layer F.Fab) (width 0.1))
     (fp_line (start 0 -1.27) (end 3.81 -1.27) (layer F.Fab) (width 0.1))
-    (fp_line (start 3.81 -1.27) (end 3.81 6.35) (layer F.Fab) (width 0.1))
-    (fp_line (start 3.81 6.35) (end -1.27 6.35) (layer F.Fab) (width 0.1))
-    (fp_line (start -1.27 6.35) (end -1.27 0) (layer F.Fab) (width 0.1))
-    (fp_line (start -1.27 0) (end 0 -1.27) (layer F.Fab) (width 0.1))
-    (fp_line (start -1.33 6.41) (end 3.87 6.41) (layer F.SilkS) (width 0.12))
-    (fp_line (start -1.33 1.27) (end -1.33 6.41) (layer F.SilkS) (width 0.12))
-    (fp_line (start 3.87 -1.33) (end 3.87 6.41) (layer F.SilkS) (width 0.12))
-    (fp_line (start -1.33 1.27) (end 1.27 1.27) (layer F.SilkS) (width 0.12))
-    (fp_line (start 1.27 1.27) (end 1.27 -1.33) (layer F.SilkS) (width 0.12))
-    (fp_line (start 1.27 -1.33) (end 3.87 -1.33) (layer F.SilkS) (width 0.12))
-    (fp_line (start -1.33 0) (end -1.33 -1.33) (layer F.SilkS) (width 0.12))
-    (fp_line (start -1.33 -1.33) (end 0 -1.33) (layer F.SilkS) (width 0.12))
-    (fp_line (start -1.8 -1.8) (end -1.8 6.85) (layer F.CrtYd) (width 0.05))
-    (fp_line (start -1.8 6.85) (end 4.35 6.85) (layer F.CrtYd) (width 0.05))
-    (fp_line (start 4.35 6.85) (end 4.35 -1.8) (layer F.CrtYd) (width 0.05))
-    (fp_line (start 4.35 -1.8) (end -1.8 -1.8) (layer F.CrtYd) (width 0.05))
-    (fp_text user %R (at 1.27 2.54 90) (layer F.Fab)
-      (effects (font (size 1 1) (thickness 0.15)))
-    )
+    (pad 6 thru_hole oval (at 2.54 5.08) (size 1.7 1.7) (drill 1) (layers *.Cu *.Mask)
+      (net 1 GND))
+    (pad 5 thru_hole oval (at 0 5.08) (size 1.7 1.7) (drill 1) (layers *.Cu *.Mask)
+      (net 1 GND))
+    (pad 4 thru_hole oval (at 2.54 2.54) (size 1.7 1.7) (drill 1) (layers *.Cu *.Mask)
+      (net 47 /BOOT1))
+    (pad 3 thru_hole oval (at 0 2.54) (size 1.7 1.7) (drill 1) (layers *.Cu *.Mask)
+      (net 46 /BOOT0))
+    (pad 2 thru_hole oval (at 2.54 0) (size 1.7 1.7) (drill 1) (layers *.Cu *.Mask)
+      (net 7 VCC))
     (pad 1 thru_hole rect (at 0 0) (size 1.7 1.7) (drill 1) (layers *.Cu *.Mask)
       (net 7 VCC))
-    (pad 2 thru_hole oval (at 2.54 0) (size 1.7 1.7) (drill 1) (layers *.Cu *.Mask)
-      (net 7 VCC))
-    (pad 3 thru_hole oval (at 0 2.54) (size 1.7 1.7) (drill 1) (layers *.Cu *.Mask)
-      (net 46 /BOOT0))
-    (pad 4 thru_hole oval (at 2.54 2.54) (size 1.7 1.7) (drill 1) (layers *.Cu *.Mask)
-      (net 47 /BOOT1))
-    (pad 5 thru_hole oval (at 0 5.08) (size 1.7 1.7) (drill 1) (layers *.Cu *.Mask)
-      (net 1 GND))
-    (pad 6 thru_hole oval (at 2.54 5.08) (size 1.7 1.7) (drill 1) (layers *.Cu *.Mask)
-      (net 1 GND))
-    (model ${KISYS3DMOD}/Connector_PinHeader_2.54mm.3dshapes/PinHeader_2x03_P2.54mm_Vertical.wrl
-      (at (xyz 0 0 0))
-      (scale (xyz 1 1 1))
+    (model ${KISYS3DMOD}/Pin_Headers.3dshapes/Pin_Header_Straight_2x03_Pitch2.54mm.wrl
+      (at (xyz 0 0 0))
+      (scale (xyz 1 1 1))

Commit message: initial commit
Parts:
- C2, C3, C4, C5, R14, R15, R6, R7, U1, U2: moved to F.Cu
- D2: moved to B.Cu
- moved U3 87.6 mm to (104.7, 133.3)
- moved C4 79.6 mm to (167.6, 114.5)
- moved Y2 79.6 mm to (171.6, 112.8), turned to 0 degrees
- moved C5 77.9 mm to (161.2, 121.4)
- moved C2 75.7 mm to (167.6, 111.7), turned to 0 degrees
- moved C3 74.5 mm to (156.8, 125.6), turned to 0 degrees
- moved J13 74.0 mm to (123.0, 132.7)
- moved R2 70.0 mm to (155.5, 119.9), turned to 0 degrees
- moved J8 63.8 mm to (131.3, 121.0), turned to 0 degrees
- moved R6 63.1 mm to (167.2, 103.1), turned to 0 degrees
- moved R7 62.5 mm to (155.5, 117.0), turned to 0 degrees
- moved R3 60.5 mm to (110.5, 132.5), turned to 0 degrees
- moved R15 59.3 mm to (172.9, 103.1), turned to 0 degrees
- moved R9 52.0 mm to (150.4, 112.8)
- moved Y1 47.6 mm to (105.8, 127.7), turned to 0 degrees
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Routing:
- net GND: track 102.2 -> 0.00 mm, vias 3 -> 0
- net VCC: track 59.6 -> 0.00 mm
- net Net-(J2-Pad3): track 49.7 -> 0.00 mm
- net Net-(J2-Pad2): track 46.1 -> 0.00 mm
- net Net-(D2-Pad23): track 38.2 -> 0.00 mm, vias 1 -> 0
- net Net-(J12-Pad1): track 37.5 -> 0.00 mm
- net Net-(D2-Pad22): track 36.1 -> 0.00 mm, vias 1 -> 0
- net Net-(C4-Pad1): track 34.6 -> 0.00 mm, vias 1 -> 0
- net Net-(J14-Pad2): track 33.0 -> 0.00 mm
- net Net-(C5-Pad1): track 28.8 -> 0.00 mm, vias 1 -> 0
- net /R: track 24.3 -> 0.00 mm, vias 1 -> 0
- net Net-(C2-Pad1): track 20.1 -> 0.00 mm
- net /3v3_STLink: track 14.4 -> 0.00 mm
- net Net-(C3-Pad1): track 14.3 -> 0.00 mm
- net /i2c1_scl: track 13.8 -> 0.00 mm
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